Commit message: Add necessary URDF for gazebo.

File: src/my_bot/description/gazebo_control.xacro (robot description, xacro)
@@ -4,6 +4,6 @@
     <plugin name="diff_drive" filename="libgazebo_ros_diff_drive.so"> <!-- filename of ROS plugin -->
       <!-- Wheel information -->
-      <left_joint>left_wheel_joint</left_joint>
-      <right_joint>right_wheel_joint</right_joint>
+      <left_joint>left_front_wheel_joint</left_joint>
+      <right_joint>right_front_wheel_joint</right_joint>
       <wheel_separation>0.35</wheel_separation>
       <wheel_diameter>0.1</wheel_diameter>

File: src/my_bot/description/robot_core.xacro (robot description, xacro)
@@ -19,13 +19,13 @@
       <material name="white" />
     </visual>
-    <!-- <collision>
-        <origin xyz="0.15 0 0.075" />
+    <collision>
+        <origin xyz="0.375 0 0.075" />
         <geometry>
-          <box size="0.3 0.3 0.15" />
+          <box size="0.75 0.3 0.15" />
         </geometry>
-      </collision>
-      <xacro:inertial_box mass="0.5" x="0.3" y="0.3" z="0.15">
-        <origin xyz="0.15 0 0.075" rpy="0 0 0" />
-      </xacro:inertial_box> -->
+    </collision>
+    <xacro:inertial_box mass="0.5" x="0.375" y="0" z="0.075">
+      <origin xyz="0.375 0 0.075" rpy="0 0 0" />
+    </xacro:inertial_box>
   </link>
   <gazebo reference="chassis">
@@ -40,13 +40,16 @@
       <material name="blue" />
     </visual>
-    <!-- <collision>
+    <collision>
       <geometry>
-        <cylinder radius="0.05" length="0.04" />
+        <cylinder radius="0.075" length="0.04" />
       </geometry>
     </collision>
-    <xacro:inertial_cylinder mass="0.1" length="0.04" radius="0.05">
+    <xacro:inertial_cylinder mass="0.1" length="0.04" radius="0.075">
       <origin xyz="0 0 0" rpy="0 0 0" />
-    </xacro:inertial_cylinder> -->
+    </xacro:inertial_cylinder>
   </link>
+  <gazebo reference="left_back_wheel">
+    <material>Gazebo/Blue</material>
+  </gazebo>
   <!-- Front Left Wheel -->
   <link name="left_front_wheel">
@@ -57,13 +60,16 @@
       <material name="blue" />
     </visual>
-    <!-- <collision>
+    <collision>
       <geometry>
-        <cylinder radius="0.05" length="0.04" />
+        <cylinder radius="0.075" length="0.04" />
       </geometry>
     </collision>
     <xacro:inertial_cylinder mass="0.1" length="0.04" radius="0.05">
       <origin xyz="0 0 0" rpy="0 0 0" />
-    </xacro:inertial_cylinder> -->
+    </xacro:inertial_cylinder>
   </link>
+  <gazebo reference="left_front_wheel">
+    <material>Gazebo/Blue</material>
+  </gazebo>
   <!-- Back Right Wheel -->
   <link name="right_back_wheel">
@@ -74,13 +80,16 @@
       <material name="blue" />
     </visual>
-    <!-- <collision>
+    <collision>
       <geometry>
-        <cylinder radius="0.05" length="0.04" />
+        <cylinder radius="0.075" length="0.04" />
       </geometry>
     </collision>
     <xacro:inertial_cylinder mass="0.1" length="0.04" radius="0.05">
       <origin xyz="0 0 0" rpy="0 0 0" />
-    </xacro:inertial_cylinder> -->
+    </xacro:inertial_cylinder>
   </link>
+  <gazebo reference="right_back_wheel">
+    <material>Gazebo/Blue</material>
+  </gazebo>
   <!-- Front Right Wheel -->
   <link name="right_front_wheel">
@@ -91,13 +100,16 @@
       <material name="blue" />
     </visual>
-    <!-- <collision>
-        <geometry>
-          <cylinder radius="0.05" length="0.04" />
-        </geometry>
-      </collision>
-      <xacro:inertial_cylinder mass="0.1" length="0.04" radius="0.05">
-        <origin xyz="0 0 0" rpy="0 0 0" />
-      </xacro:inertial_cylinder> -->
+    <collision>
+      <geometry>
+        <cylinder radius="0.075" length="0.04" />
+      </geometry>
+    </collision>
+    <xacro:inertial_cylinder mass="0.1" length="0.04" radius="0.05">
+      <origin xyz="0 0 0" rpy="0 0 0" />
+    </xacro:inertial_cylinder>
   </link>
+  <gazebo reference="right_front_wheel">
+    <material>Gazebo/Blue</material>
+  </gazebo>
   <!-- ====================== Joints ======================== -->
   <!-- Chassis Joint -->
@@ -141,5 +153,5 @@
     <!-- transform from parent link to child link -->
     <!-- joint is located at origin of child link -->
-    <origin xyz="${wheel_from_center} -0.175 0" rpy="-${pi/2} 0 0" />
+    <origin xyz="${wheel_from_center} -0.175 0" rpy="${pi/2} 0 0" />
     <!-- axis of rotation; takes normalized vector of direction to rotate around -->
     <axis xyz="0 0 -1" />
