Commit message: Use constants for dimensions.

File: src/my_bot/description/robot_core.xacro (robot description, xacro)
@@ -4,27 +4,40 @@
   <xacro:include filename="colours.xacro" />
   <!-- ====================== Constants ======================== -->
-  <xacro:property name="wheel_from_center" value="0.2"/>
-  <!-- ====================== Links ======================== -->
+  <!-- Using REP 103 here. -njreichert -->
+  <xacro:property name="chassis_length" value="0.75" />
+  <xacro:property name="chassis_width" value="0.3" />
+  <xacro:property name="chassis_height" value="0.15" />
+  <xacro:property name="wheel_chassis_buffer_len" value="0.005" />
+  <xacro:property name="wheel_x_spacing" value="0.2" />
+  <xacro:property name="wheel_y_spacing" value="${(chassis_width / 2) + (wheel_length / 2) + wheel_chassis_buffer_len}"/>
+  <xacro:property name="wheel_radius" value="0.075" />
+  <xacro:property name="wheel_length" value="0.04" />
   <!-- Base Link -->
   <link name="base_link">
   </link>
   <!-- Chassis -->
+  <joint name="chassis_joint" type="fixed">
+    <parent link="base_link" />
+    <child link="chassis" />
+    <!-- separation distance between base_link (middle of chassis) and chassis origin -->
+    <origin xyz="-${chassis_length / 2} 0 0" />
+  </joint>
   <link name="chassis">
     <visual>
       <!-- shift box forward so chassis link origin is centered at back bottom -->
-      <origin xyz="0.375 0 0.075" />
+      <origin xyz="${chassis_length / 2} 0 ${chassis_height / 2}" />
       <geometry>
-        <box size="0.75 0.3 0.15" />
+        <box size="${chassis_length} ${chassis_width} ${chassis_height}" />
       </geometry>
       <material name="white" />
     </visual>
     <collision>
-        <origin xyz="0.375 0 0.075" />
+        <origin xyz="${chassis_length / 2} 0 ${chassis_height / 2}" />
         <geometry>
-          <box size="0.75 0.3 0.15" />
+          <box size="${chassis_length} ${chassis_width} ${chassis_height}" />
         </geometry>
     </collision>
-    <xacro:inertial_box mass="0.5" x="0.375" y="0" z="0.075">
-      <origin xyz="0.375 0 0.075" rpy="0 0 0" />
+    <xacro:inertial_box mass="0.5" x="${chassis_length / 2}" y="0" z="${chassis_height / 2}">
+      <origin xyz="${chassis_length / 2} 0 ${chassis_height / 2}" rpy="0 0 0" />
     </xacro:inertial_box>
   </link>
@@ -33,8 +46,17 @@
   </gazebo>
   <!-- Back Left Wheel -->
+  <joint name="left_back_wheel_joint" type="continuous">
+    <parent link="base_link" />
+    <child link="left_back_wheel" />
+    <!-- transform from parent link to child link -->
+    <!-- joint is located at origin of child link -->
+    <origin xyz="-${wheel_x_spacing} ${wheel_y_spacing} 0" rpy="-${pi/2} 0 0" />
+    <!-- axis of rotation; takes normalized vector of direction to rotate around -->
+    <axis xyz="0 0 1" />
+  </joint>
   <link name="left_back_wheel">
     <visual>
       <geometry>
-        <cylinder radius="0.075" length="0.04" />
+        <cylinder radius="${wheel_radius}" length="${wheel_length}" />
       </geometry>
       <material name="blue" />
@@ -42,8 +64,8 @@
     <collision>
       <geometry>
-        <cylinder radius="0.075" length="0.04" />
+        <cylinder radius="${wheel_radius}" length="${wheel_length}" />
       </geometry>
     </collision>
-    <xacro:inertial_cylinder mass="0.1" length="0.04" radius="0.075">
+    <xacro:inertial_cylinder mass="0.1" length="${wheel_length}" radius="${wheel_radius}">
       <origin xyz="0 0 0" rpy="0 0 0" />
     </xacro:inertial_cylinder>
@@ -53,8 +75,17 @@
   </gazebo>
   <!-- Front Left Wheel -->
+  <joint name="left_front_wheel_joint" type="continuous">
+    <parent link="base_link" />
+    <child link="left_front_wheel" />
+    <!-- transform from parent link to child link -->
+    <!-- joint is located at origin of child link -->
+    <origin xyz="${wheel_x_spacing} ${wheel_y_spacing} 0" rpy="-${pi/2} 0 0" />
+    <!-- axis of rotation; takes normalized vector of direction to rotate around -->
+    <axis xyz="0 0 1" />
+  </joint>
   <link name="left_front_wheel">
     <visual>
       <geometry>
-        <cylinder radius="0.075" length="0.04" />
+        <cylinder radius="${wheel_radius}" length="${wheel_length}" />
       </geometry>
       <material name="blue" />
@@ -62,8 +93,8 @@
     <collision>
       <geometry>
-        <cylinder radius="0.075" length="0.04" />
+        <cylinder radius="${wheel_radius}" length="${wheel_length}" />
       </geometry>
     </collision>
-    <xacro:inertial_cylinder mass="0.1" length="0.04" radius="0.05">
+    <xacro:inertial_cylinder mass="0.1" length="${wheel_length}" radius="${wheel_radius}">
       <origin xyz="0 0 0" rpy="0 0 0" />
     </xacro:inertial_cylinder>
@@ -73,8 +104,14 @@
   </gazebo>
   <!-- Back Right Wheel -->
+  <joint name="right_back_wheel_joint" type="continuous">
+    <parent link="base_link" />
+    <child link="right_back_wheel" />
+    <origin xyz="-${wheel_x_spacing} -${wheel_y_spacing} 0" rpy="${pi/2} 0 0" />
+    <axis xyz="0 0 -1" />
+  </joint>
   <link name="right_back_wheel">
     <visual>
       <geometry>
-        <cylinder radius="0.075" length="0.04" />
+        <cylinder radius="${wheel_radius}" length="${wheel_length}" />
       </geometry>
       <material name="blue" />
@@ -82,8 +119,8 @@
     <collision>
       <geometry>
-        <cylinder radius="0.075" length="0.04" />
+        <cylinder radius="${wheel_radius}" length="${wheel_length}" />
       </geometry>
     </collision>
-    <xacro:inertial_cylinder mass="0.1" length="0.04" radius="0.05">
+    <xacro:inertial_cylinder mass="0.1" length="${wheel_length}" radius="${wheel_radius}">
       <origin xyz="0 0 0" rpy="0 0 0" />
     </xacro:inertial_cylinder>
@@ -93,8 +130,17 @@
   </gazebo>
   <!-- Front Right Wheel -->
+  <joint name="right_front_wheel_joint" type="continuous">
+    <parent link="base_link" />
+    <child link="right_front_wheel" />
+    <!-- transform from parent link to child link -->
+    <!-- joint is located at origin of child link -->
+    <origin xyz="${wheel_x_spacing} -${wheel_y_spacing} 0" rpy="${pi/2} 0 0" />
+    <!-- axis of rotation; takes normalized vector of direction to rotate around -->
+    <axis xyz="0 0 -1" />
+  </joint>
   <link name="right_front_wheel">
     <visual>
       <geometry>
-        <cylinder radius="0.075" length="0.04" />
+        <cylinder radius="${wheel_radius}" length="${wheel_length}" />
       </geometry>
       <material name="blue" />
@@ -102,8 +148,8 @@
     <collision>
       <geometry>
-        <cylinder radius="0.075" length="0.04" />
+        <cylinder radius="${wheel_radius}" length="${wheel_length}" />
       </geometry>
     </collision>
-    <xacro:inertial_cylinder mass="0.1" length="0.04" radius="0.05">
+    <xacro:inertial_cylinder mass="0.1" length="${wheel_length}" radius="${wheel_radius}">
       <origin xyz="0 0 0" rpy="0 0 0" />
     </xacro:inertial_cylinder>
@@ -112,76 +158,3 @@
     <material>Gazebo/Blue</material>
   </gazebo>
-  <!-- ====================== Joints ======================== -->
-  <!-- Chassis Joint -->
-  <joint name="chassis_joint" type="fixed">
-    <parent link="base_link" />
-    <child link="chassis" />
-    <!-- separation distance between base_link (middle of chassis) and chassis origin -->
-    <origin xyz="-0.375 0 0" />
-  </joint>
-  <!-- Back Left Wheel Joint -->
-  <joint name="left_back_wheel_joint" type="continuous">
-    <parent link="base_link" />
-    <child link="left_back_wheel" />
-    <!-- transform from parent link to child link -->
-    <!-- joint is located at origin of child link -->
-    <origin xyz="-${wheel_from_center} 0.175 0" rpy="-${pi/2} 0 0" />
-    <!-- axis of rotation; takes normalized vector of direction to rotate around -->
-    <axis xyz="0 0 1" />
-  </joint>
-  <!-- Front Left Wheel Joint -->
-  <joint name="left_front_wheel_joint" type="continuous">
-    <parent link="base_link" />
-    <child link="left_front_wheel" />
-    <!-- transform from parent link to child link -->
-    <!-- joint is located at origin of child link -->
-    <origin xyz="${wheel_from_center} 0.175 0" rpy="-${pi/2} 0 0" />
-    <!-- axis of rotation; takes normalized vector of direction to rotate around -->
-    <axis xyz="0 0 1" />
-  </joint>
-  <!-- Back Right Wheel Joint -->
-  <joint name="right_back_wheel_joint" type="continuous">
-    <parent link="base_link" />
-    <child link="right_back_wheel" />
-    <origin xyz="-${wheel_from_center} -0.175 0" rpy="${pi/2} 0 0" />
-    <axis xyz="0 0 -1" />
-  </joint>
-  <!-- Front Right Wheel Joint -->
-  <joint name="right_front_wheel_joint" type="continuous">
-    <parent link="base_link" />
-    <child link="right_front_wheel" />
-    <!-- transform from parent link to child link -->
-    <!-- joint is located at origin of child link -->
-    <origin xyz="${wheel_from_center} -0.175 0" rpy="${pi/2} 0 0" />
-    <!-- axis of rotation; takes normalized vector of direction to rotate around -->
-    <axis xyz="0 0 -1" />
-  </joint>
-  <!-- Caster Wheel -->
-  <!-- <joint name="caster_wheel_joint" type="fixed">
-    <parent link="chassis" />
-    <child link="caster_wheel" />
-    <origin xyz="0.24 0 0" />
-  </joint> -->
-  <!-- <link name="caster_wheel">
-    <visual>
-      <geometry>
-        <sphere radius="0.05" />
-      </geometry>
-      <material name="black" />
-    </visual>
-    <collision>
-      <geometry>
-        <sphere radius="0.05" />
-      </geometry>
-    </collision>
-    <xacro:inertial_sphere mass="0.1" radius="0.05">
-      <origin xyz="0 0 0" rpy="0 0 0" />
-    </xacro:inertial_sphere>
-  </link> -->
-  <!--
-  <gazebo reference="caster_wheel">
-    <material>Gazebo/Black</material>
-    <mu1 value="0.001"/>
-    <mu2 value="0.001"/>
-  </gazebo> -->
 </robot>

Commit message: Add friction to drive base.

File: src/my_bot/description/robot_core.xacro (robot description, xacro)
@@ -3,4 +3,5 @@
   <xacro:include filename="inertial_macros.xacro" />
   <xacro:include filename="colours.xacro" />
+  <!-- "TODO:" Still need to look at the inertia macros to make sure they are defined properly. -njreichert -->
   <!-- ====================== Constants ======================== -->
   <!-- Using REP 103 here. -njreichert -->
@@ -13,4 +14,5 @@
   <xacro:property name="wheel_radius" value="0.075" />
   <xacro:property name="wheel_length" value="0.04" />
+  <xacro:property name="wheel_friction" value="0.8" />
   <!-- Base Link -->
   <link name="base_link">
@@ -66,4 +68,14 @@
         <cylinder radius="${wheel_radius}" length="${wheel_length}" />
       </geometry>
+      <surface>
+        <friction>
+          <ode>
+            <mu>${wheel_friction}</mu>
+            <mu2>${wheel_friction}</mu2>
+            <slip1>0.0</slip1>
+            <slip2>0.0</slip2>
+          </ode>
+        </friction>
+      </surface>
     </collision>
     <xacro:inertial_cylinder mass="0.1" length="${wheel_length}" radius="${wheel_radius}">
@@ -73,4 +85,6 @@
   <gazebo reference="left_back_wheel">
     <material>Gazebo/Blue</material>
+    <mu1>${wheel_friction}</mu1>
+    <mu2>${wheel_friction}</mu2>
   </gazebo>
   <!-- Front Left Wheel -->
@@ -95,4 +109,14 @@
         <cylinder radius="${wheel_radius}" length="${wheel_length}" />
       </geometry>
+      <surface>
+        <friction>
+          <ode>
+            <mu>${wheel_friction}</mu>
+            <mu2>${wheel_friction}</mu2>
+            <slip1>0.0</slip1>
+            <slip2>0.0</slip2>
+          </ode>
+        </friction>
+      </surface>
     </collision>
     <xacro:inertial_cylinder mass="0.1" length="${wheel_length}" radius="${wheel_radius}">
@@ -102,4 +126,6 @@
   <gazebo reference="left_front_wheel">
     <material>Gazebo/Blue</material>
+    <mu1>${wheel_friction}</mu1>
+    <mu2>${wheel_friction}</mu2>
   </gazebo>
   <!-- Back Right Wheel -->
@@ -121,4 +147,14 @@
         <cylinder radius="${wheel_radius}" length="${wheel_length}" />
       </geometry>
+      <surface>
+        <friction>
+          <ode>
+            <mu>${wheel_friction}</mu>
+            <mu2>${wheel_friction}</mu2>
+            <slip1>0.0</slip1>
+            <slip2>0.0</slip2>
+          </ode>
+        </friction>
+      </surface>
     </collision>
     <xacro:inertial_cylinder mass="0.1" length="${wheel_length}" radius="${wheel_radius}">
@@ -128,4 +164,6 @@
   <gazebo reference="right_back_wheel">
     <material>Gazebo/Blue</material>
+    <mu1>${wheel_friction}</mu1>
+    <mu2>${wheel_friction}</mu2>
   </gazebo>
   <!-- Front Right Wheel -->
@@ -150,4 +188,14 @@
         <cylinder radius="${wheel_radius}" length="${wheel_length}" />
       </geometry>
+      <surface>
+        <friction>
+          <ode>
+            <mu>${wheel_friction}</mu>
+            <mu2>${wheel_friction}</mu2>
+            <slip1>0.0</slip1>
+            <slip2>0.0</slip2>
+          </ode>
+        </friction>
+      </surface>
     </collision>
     <xacro:inertial_cylinder mass="0.1" length="${wheel_length}" radius="${wheel_radius}">
@@ -157,4 +205,6 @@
   <gazebo reference="right_front_wheel">
     <material>Gazebo/Blue</material>
+    <mu1>${wheel_friction}</mu1>
+    <mu2>${wheel_friction}</mu2>
   </gazebo>
 </robot>
