Commit message: Add ros2_control demo example. TODO: add PWM motor controller code to example, clean up launch files, etc...

File: src/my_bot/description/robot.urdf.xacro (robot description, xacro)
@@ -1,6 +1,9 @@
 <?xml version="1.0"?>
 <robot xmlns:xacro="http://www.ros.org/wiki/xacro" name="robot">
+    <xacro:arg name="prefix" default="" />
+    <xacro:arg name="use_mock_hardware" default="false" />
     <xacro:include filename="robot_core.xacro" />
     <!-- <xacro:include filename="gazebo_control.xacro"/> -->
     <xacro:include filename="ros2_control.xacro" />
+    <xacro:diffbot_ros2_control name="DiffBot" prefix="$(arg prefix)" use_mock_hardware="$(arg use_mock_hardware)" />
 </robot>

File: src/my_bot/description/ros2_control.xacro (robot description, xacro)
@@ -1,41 +1,53 @@
 <?xml version="1.0"?>
 <robot xmlns:xacro="http://www.ros.org/wiki/xacro">
-	<ros2_control name="GazeboSystem" type="system">
-		<hardware>
-			<plugin>gazebo_ros2_control/GazeboSystem</plugin>
-		</hardware>
-		<joint name="left_front_wheel_joint">
-			<command_interface name="velocity">
-				<param name="min">-10</param>
-				<param name="max">10</param>
-			</command_interface>
-			<state_interface name="velocity" />
-			<state_interface name="position" />
-		</joint>
-		<joint name="right_front_wheel_joint">
-			<command_interface name="velocity">
-				<param name="min">-10</param>
-				<param name="max">10</param>
-			</command_interface>
-			<state_interface name="velocity" />
-			<state_interface name="position" />
-		</joint>
-		<joint name="left_back_wheel_joint">
-			<command_interface name="velocity">
-				<param name="min">-10</param>
-				<param name="max">10</param>
-			</command_interface>
-			<state_interface name="velocity" />
-			<state_interface name="position" />
-		</joint>
-		<joint name="right_back_wheel_joint">
-			<command_interface name="velocity">
-				<param name="min">-10</param>
-				<param name="max">10</param>
-			</command_interface>
-			<state_interface name="velocity" />
-			<state_interface name="position" />
-		</joint>
-	</ros2_control>
+	<xacro:macro name="diffbot_ros2_control" params="name prefix use_mock_hardware">
+		<ros2_control name="${name}" type="system">
+			<xacro:unless value="${use_mock_hardware}">
+				<hardware>
+				<plugin>ros2_control_demo_example_2/DiffBotSystemHardware</plugin>
+				<param name="example_param_hw_start_duration_sec">0</param>
+				<param name="example_param_hw_stop_duration_sec">3.0</param>
+				</hardware>
+			</xacro:unless>
+			<xacro:if value="${use_mock_hardware}">
+				<hardware>
+				<plugin>mock_components/GenericSystem</plugin>
+				<param name="calculate_dynamics">true</param>
+				</hardware>
+			</xacro:if>
+			<joint name="left_front_wheel_joint">
+				<command_interface name="velocity">
+					<param name="min">-10</param>
+					<param name="max">10</param>
+				</command_interface>
+				<state_interface name="position" />
+				<state_interface name="velocity" />
+			</joint>
+			<joint name="right_front_wheel_joint">
+				<command_interface name="velocity">
+					<param name="min">-10</param>
+					<param name="max">10</param>
+				</command_interface>
+				<state_interface name="position" />
+				<state_interface name="velocity" />
+			</joint>
+			<joint name="left_back_wheel_joint">
+				<command_interface name="velocity">
+					<param name="min">-10</param>
+					<param name="max">10</param>
+				</command_interface>
+				<state_interface name="position" />
+				<state_interface name="velocity" />
+			</joint>
+			<joint name="right_back_wheel_joint">
+				<command_interface name="velocity">
+					<param name="min">-10</param>
+					<param name="max">10</param>
+				</command_interface>
+				<state_interface name="position" />
+				<state_interface name="velocity" />
+			</joint>
+		</ros2_control>
+	</xacro:macro>
 	<gazebo>
 		<!-- This plugin has its own Controller Manager. -->
